Commit message: updated files

File: aigo_urdf/urdf/aigo.urdf (robot description, URDF)
Before this commit: robot aigo, 6 links, 5 joints
Links:
- added link gps
Joints:
- added joint gps_to_base_link: type fixed, parent base_link, child gps, origin xyz=0 0 0 rpy=0 0 0

Commit message: attatched new sensor

File: aigo_urdf/urdf/aigo.urdf (robot description, URDF)
Before this commit: robot aigo, 8 links, 7 joints
Links:
- removed link imu_frame
- added link imu_link
Joints:
- joint imu_to_base_link: child imu_frame -> imu_link
